Commit message: Update kitten.urdf

File: vehicle_model/kitten.urdf (robot description, URDF)
Before this commit: robot pacifica_structure, 10 links, 9 joints
Links:
- removed link base
- removed link map
- added link base_footprint, mass 2242.0; collision mesh filename=../urdf/meshes/pacifica_18/body_collision.stl scale=0.96 0.96 0.96; visual mesh filename=../urdf/meshes/pacifica_18/body.dae scale=0.96 0.96 0.96
- added link velodyne_frame
- link wheel_fl: geometry collision cylinder length=0.25 radius=0.365; visual mesh filename=../urdf/meshes/pacifica_18/wheel.dae
- link wheel_fr: geometry collision cylinder length=0.25 radius=0.365; visual mesh filename=../urdf/meshes/pacifica_18/wheel.dae
- link wheel_rl: geometry collision cylinder length=0.25 radius=0.365; visual mesh filename=../urdf/meshes/pacifica_18/wheel.dae
- link wheel_rr: geometry collision cylinder length=0.25 radius=0.365; visual mesh filename=../urdf/meshes/pacifica_18/wheel.dae
Joints:
- removed joint base
- added joint base_link_joint: type fixed, parent velodyne_frame, child base_footprint, origin xyz=0.54 0 -1.435 rpy=0 0 0
- joint cam_00_to_velo_joint: parent map -> velodyne_frame
- joint cam_01_to_velo_joint: parent map -> velodyne_frame
- joint steer_fl_joint: parent base -> base_footprint
- joint steer_fr_joint: parent base -> base_footprint
- joint wheel_rl_joint: parent base -> base_footprint
- joint wheel_rr_joint: parent base -> base_footprint
