Commit message: Update vehicle.urdf

File: vehicle_model/vehicle.urdf (robot description, URDF)
Before this commit: robot lexus_rx_450h, 1 links, 0 joints
Links:
- link base: geometry collision box size=5.5 2.25 2; visual mesh filename=package://vehicle_model/meshes/lc.stl scale=1.0 1.0 1.0

Commit message: Update vehicle.urdf

File: vehicle_model/vehicle.urdf (robot description, URDF)
Before this commit: robot lexus_rx_450h, 1 links, 0 joints
Links:
- link base: geometry collision box size=5.5 2.25 2; visual mesh filename=package://vehicle_model/meshes/lc.dae scale=1.0 1.0 1.0

Commit message: Update vehicle.urdf

File: vehicle_model/vehicle.urdf (robot description, URDF)
Before this commit: robot vehicle, 1 links, 0 joints
Links:
- link base: geometry collision box size=5.5 2.25 2; visual mesh filename=https://github.com/allenwang-git/vehicle-model/blob/main/ve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 scale=1.0 1.0 1.0

Commit message: Update vehicle.urdf

File: vehicle_model/vehicle.urdf (robot description, URDF)
Before this commit: robot vehicle, 1 links, 0 joints
Links:
- added link map
- link base: geometry collision box size=5.5 2.25 2; visual mesh filename=./meshes/lc.dae scale=1.0 1.0 1.0
